Commit message: urdf_update

File: ROS/osr_gazebo/urdf/gazebo.urdf.xacro (robot description, xacro)
@@ -49,6 +49,10 @@
     <joint name="front_wheel_joint_R">
       <command_interface name="position">
-        <param name="min">-70</param>
-        <param name="max">70</param>
+        <param name="min">-5</param>
+        <param name="max">5</param>
+      </command_interface>
+      <command_interface name="velocity">
+        <param name="min">-0.1</param>
+        <param name="max">0.1</param>
       </command_interface>
       <state_interface name="position"/>
@@ -58,6 +62,10 @@
     <joint name="front_wheel_joint_L">
       <command_interface name="position">
-        <param name="min">-70</param>
-        <param name="max">70</param>
+        <param name="min">-5</param>
+        <param name="max">5</param>
+      </command_interface>
+      <command_interface name="velocity">
+        <param name="min">-0.1</param>
+        <param name="max">0.1</param>
       </command_interface>
       <state_interface name="position"/>
@@ -66,7 +74,11 @@
     </joint>
     <joint name="rear_wheel_joint_R">
-       <command_interface name="position">
-        <param name="min">-70</param>
-        <param name="max">70</param>
+      <command_interface name="position">
+        <param name="min">-5</param>
+        <param name="max">5</param>
+      </command_interface>
+      <command_interface name="velocity">
+        <param name="min">-0.1</param>
+        <param name="max">0.1</param>
       </command_interface>
       <state_interface name="position"/>
@@ -76,6 +88,10 @@
     <joint name="rear_wheel_joint_L">
       <command_interface name="position">
-        <param name="min">-70</param>
-        <param name="max">70</param>
+        <param name="min">-5</param>
+        <param name="max">5</param>
+      </command_interface>
+      <command_interface name="velocity">
+        <param name="min">-0.1</param>
+        <param name="max">0.1</param>
       </command_interface>
       <state_interface name="position"/>

File: ROS/osr_gazebo/urdf/insert_transmission.urdf.xacro (robot description, xacro)
@@ -4,10 +4,10 @@
         <transmission name="${name}_tran">
             <type>transmission_interface/SimpleTransmission</type>
-            <joint name="${name}" >
-                <hardwareInterface>hardware_interface/EffortJointInterface</hardwareInterface>
+            <joint name="${name}">
+                <hardwareInterface>EffortJointInterface</hardwareInterface>  <!-- Updated for ROS2 -->
                 <mechanicalReduction>1</mechanicalReduction>
             </joint>
             <actuator name="${name}_motor">
-                <hardwareInterface>hardware_interface/EffortJointInterface</hardwareInterface>
+                <hardwareInterface>EffortJointInterface</hardwareInterface>  <!-- Updated for ROS2 -->
                 <mechanicalReduction>1</mechanicalReduction>
             </actuator>
@@ -17,10 +17,10 @@
         <transmission name="${name}_tran">
             <type>transmission_interface/SimpleTransmission</type>
-            <joint name="${name}" >
-                <hardwareInterface>hardware_interface/PositionJointInterface</hardwareInterface>
+            <joint name="${name}">
+                <hardwareInterface>PositionJointInterface</hardwareInterface>  <!-- Updated for ROS2 -->
                 <mechanicalReduction>1</mechanicalReduction>
             </joint>
             <actuator name="${name}_motor">
-                <hardwareInterface>hardware_interface/PositionJointInterface</hardwareInterface>
+                <hardwareInterface>PositionJointInterface</hardwareInterface>  <!-- Updated for ROS2 -->
                 <mechanicalReduction>1</mechanicalReduction>
             </actuator>
@@ -30,10 +30,10 @@
         <transmission name="${name}_tran">
             <type>transmission_interface/SimpleTransmission</type>
-            <joint name="${name}" >
-                <hardwareInterface>hardware_interface/VelocityJointInterface</hardwareInterface>
+            <joint name="${name}">
+                <hardwareInterface>VelocityJointInterface</hardwareInterface>  <!-- Updated for ROS2 -->
                 <mechanicalReduction>1</mechanicalReduction>
             </joint>
             <actuator name="${name}_motor">
-                <hardwareInterface>hardware_interface/VelocityJointInterface</hardwareInterface>
+                <hardwareInterface>VelocityJointInterface</hardwareInterface>  <!-- Updated for ROS2 -->
                 <mechanicalReduction>1</mechanicalReduction>
             </actuator>

File: ROS/osr_gazebo/urdf/osr.urdf.xacro (robot description, xacro)
@@ -17,5 +17,5 @@
     </material>
     <xacro:include filename="$(find osr_gazebo)/urdf/gazebo.urdf.xacro"/>
-    <!-- <xacro:include filename="$(find osr_gazebo)/urdf/insert_transmission.urdf.xacro"/>  -->
+    <xacro:include filename="$(find osr_gazebo)/urdf/insert_transmission.urdf.xacro"/>
     <link name="base_footprint"/>
     <link name="base_link">
@@ -414,9 +414,13 @@
     <xacro:wheel prefix="left" dir="1" origin="0" prefix_1="L"/>
     <xacro:wheel prefix="right" dir="-1" origin="3.14" prefix_1="R"/>
-    <joint name="imu_joint" type="fixed">
-            <parent link="base_link"/>
-            <child link="imu_link"/>
-            <origin xyz="0 0 0" rpy="0 0 0"/>
-        </joint>
-    <link name="imu_link"></link>
+    <xacro:insert_velocity_transmission name="rear_wheel_joint_right"/>
+    <xacro:insert_velocity_transmission name="rear_wheel_joint_left"/>
+    <xacro:insert_velocity_transmission name="middle_wheel_joint_right"/>
+    <xacro:insert_velocity_transmission name="middle_wheel_joint_left"/>
+    <xacro:insert_velocity_transmission name="front_wheel_joint_right"/>
+    <xacro:insert_velocity_transmission name="front_wheel_joint_left"/>
+    <xacro:insert_position_transmission name="front_wheel_joint_R"/>
+    <xacro:insert_position_transmission name="front_wheel_joint_L"/>
+    <xacro:insert_position_transmission name="rear_wheel_joint_R"/>
+    <xacro:insert_position_transmission name="rear_wheel_joint_L"/>
 </robot>

Commit message: odom_update

File: ROS/osr_gazebo/urdf/gazebo.urdf.xacro (robot description, xacro)
@@ -10,4 +10,5 @@
         <param name="max">10</param>
       </command_interface>
+      <state_interface name="position"/>
       <state_interface name="velocity"/>
     </joint>
@@ -17,5 +18,7 @@
         <param name="max">10</param>
       </command_interface>
+      <state_interface name="position"/>
       <state_interface name="velocity"/>
+      <state_interface name="effort"/>
     </joint>
     <joint name="rear_wheel_joint_left">
@@ -24,5 +27,7 @@
         <param name="max">10</param>
       </command_interface>
+      <state_interface name="position"/>
       <state_interface name="velocity"/>
+      <state_interface name="effort"/>
     </joint>
     <joint name="rear_wheel_joint_right">
@@ -31,5 +36,7 @@
         <param name="max">10</param>
       </command_interface>
+      <state_interface name="position"/>
       <state_interface name="velocity"/>
+      <state_interface name="effort"/>
     </joint>
     <joint name="front_wheel_joint_left">
@@ -38,5 +45,7 @@
         <param name="max">10</param>
       </command_interface>
+      <state_interface name="position"/>
       <state_interface name="velocity"/>
+      <state_interface name="effort"/>
     </joint>
     <joint name="front_wheel_joint_right">
@@ -45,5 +54,7 @@
         <param name="max">10</param>
       </command_interface>
+      <state_interface name="position"/>
       <state_interface name="velocity"/>
+      <state_interface name="effort"/>
     </joint>
     <joint name="front_wheel_joint_R">
@@ -105,3 +116,23 @@
     </plugin>
   </gazebo>
+    <gazebo reference="imu_link">
+        <gravity>true</gravity>
+        <sensor name="imu_sensor" type="imu">
+        <always_on>true</always_on>
+        <update_rate>100</update_rate>
+        <visualize>true</visualize>
+        <topic>"imu"</topic>
+        <plugin filename="libgazebo_ros_imu_sensor.so" name="imu_plugin">
+            <topicName>imu</topicName>
+            <bodyName>imu_link</bodyName>
+            <updateRateHZ>100.0</updateRateHZ>
+            <gaussianNoise>0.0</gaussianNoise>
+            <xyzOffset>0 0 0</xyzOffset>
+            <rpyOffset>0 0 0</rpyOffset>
+            <frameName>imu_link</frameName>
+            <initialOrientationAsReference>false</initialOrientationAsReference>
+        </plugin>
+        <pose>0 0 0 0 0 0</pose>
+        </sensor>
+    </gazebo>
 </robot>

File: ROS/osr_gazebo/urdf/osr.urdf.xacro (robot description, xacro)
@@ -414,4 +414,10 @@
     <xacro:wheel prefix="left" dir="1" origin="0" prefix_1="L"/>
     <xacro:wheel prefix="right" dir="-1" origin="3.14" prefix_1="R"/>
+    <joint name="imu_joint" type="fixed">
+            <parent link="base_link"/>
+            <child link="imu_link"/>
+            <origin xyz="0 0 0" rpy="0 0 0"/>
+        </joint>
+    <link name="imu_link"></link>
     <xacro:insert_velocity_transmission name="rear_wheel_joint_right"/>
     <xacro:insert_velocity_transmission name="rear_wheel_joint_left"/>
