Commit message: Widen Gazebo URDF steer-joint limits to cover the angles kinematics.py commands
Closes #225

File: ROS/osr_gazebo/urdf/osr.urdf.xacro (robot description, xacro)
@@ -245,5 +245,5 @@
             <origin rpy="0 0 0" xyz="0.170113 -0.000335 0.076721"/>
             <child link="front_wheel_link_${prefix}"/>
-            <limit effort="100000.0" velocity="10" lower="-0.523599" upper="0.523599"/>
+            <limit effort="100000.0" velocity="10" lower="-1.15" upper="1.15"/>
             <axis xyz="0 0 1"/>
         </joint>
@@ -299,5 +299,5 @@
             <origin rpy="0 0 0" xyz="-0.311763 0 -0.030379"/>
             <child link="rear_wheel_link_${prefix}"/>
-            <limit effort="100000.0" velocity="3" lower="-0.523599" upper="0.523599"/>
+            <limit effort="100000.0" velocity="3" lower="-1.15" upper="1.15"/>
             <axis xyz="0 0 1"/>
         </joint>

Commit message: docs: don't refer to what was in the past

File: ROS/osr_gazebo/urdf/osr.urdf.xacro (robot description, xacro)
@@ -305,7 +305,5 @@
     <xacro:wheel_link prefix="L" dir="1" origin="1.57"/>
     <xacro:wheel_link prefix="R" dir="-1" origin="-3.14"/>
-    <!-- Wheel-ground friction. It has to be set through <gazebo reference>:
-         a <surface> block inside a URDF <collision> is dropped when the URDF is
-         converted to SDF, so it never reaches the simulator. -->
+    <!-- Wheel-ground friction -->
     <xacro:property name="wheel_mu1" value="0.7"/>
     <xacro:property name="wheel_mu2" value="0.7"/>
