Commit message: Apply Gazebo wheel friction through <gazebo reference>
The wheels' friction was set in <surface><friction> blocks inside the URDF
<collision> elements. URDF has no <surface> element, so the URDF-to-SDF
conversion drops it and the values never reached Gazebo: `gz sdf -p` of the
xacro output has 0 <mu> elements, and the wheels ran on Gazebo's default
friction (mu = 1).

Set it with <gazebo reference> mu1/mu2 on the six wheel links instead,
which the conversion carries into the SDF, from one pair of xacro
properties. Both are 0.7: the old mu2 = 0.3 only has a meaning along a
friction direction (fdir1), which was never set, so the direction it
applied in was up to the physics engine.

Co-Authored-By: Claude Opus 5.5 <noreply@anthropic.com>

File: ROS/osr_gazebo/urdf/osr.urdf.xacro (robot description, xacro)
@@ -305,5 +305,19 @@
     <xacro:wheel_link prefix="L" dir="1" origin="1.57"/>
     <xacro:wheel_link prefix="R" dir="-1" origin="-3.14"/>
+    <!-- Wheel-ground friction. It has to be set through <gazebo reference>:
+         a <surface> block inside a URDF <collision> is dropped when the URDF is
+         converted to SDF, so it never reaches the simulator. -->
+    <xacro:property name="wheel_mu1" value="0.7"/>
+    <xacro:property name="wheel_mu2" value="0.7"/>
+    <xacro:macro name="wheel_friction" params="link">
+        <gazebo reference="${link}">
+            <mu1>${wheel_mu1}</mu1>
+            <mu2>${wheel_mu2}</mu2>
+        </gazebo>
+    </xacro:macro>
     <xacro:macro name="wheel" params="prefix dir origin prefix_1">
+        <xacro:wheel_friction link="front_wheel_link_${prefix}"/>
+        <xacro:wheel_friction link="middle_wheel_link_${prefix}"/>
+        <xacro:wheel_friction link="rear_wheel_link_${prefix}"/>
         <link name="front_wheel_link_${prefix}">
             <collision>
@@ -312,12 +326,4 @@
                     <mesh filename="file://$(find osr_gazebo)/meshes/wheel.stl"/>
                 </geometry>
-                <surface>
-                    <friction>
-                        <ode>
-                            <mu>0.7</mu>
-                            <mu2>0.3</mu2>
-                        </ode>
-                    </friction>
-                </surface>
             </collision>
             <visual>
@@ -347,12 +353,4 @@
                     <mesh filename="file://$(find osr_gazebo)/meshes/wheel.stl"/>
                 </geometry>
-                <surface>
-                    <friction>
-                        <ode>
-                            <mu>0.7</mu>
-                            <mu2>0.3</mu2>
-                        </ode>
-                    </friction>
-                </surface>
             </collision>
             <visual>
@@ -382,12 +380,4 @@
                     <mesh filename="file://$(find osr_gazebo)/meshes/wheel.stl"/>
                 </geometry>
-                <surface>
-                    <friction>
-                        <ode>
-                            <mu>0.7</mu>
-                            <mu2>0.3</mu2>
-                        </ode>
-                    </friction>
-                </surface>
             </collision>
             <visual>

Commit message: Apply Gazebo wheel friction through <gazebo reference> (#230)
* Apply Gazebo wheel friction through <gazebo reference>

The wheels' friction was set in <surface><friction> blocks inside the URDF
<collision> elements. URDF has no <surface> element, so the URDF-to-SDF
conversion drops it and the values never reached Gazebo: `gz sdf -p` of the
xacro output has 0 <mu> elements, and the wheels ran on Gazebo's default
friction (mu = 1).

Set it with <gazebo reference> mu1/mu2 on the six wheel links instead,
which the conversion carries into the SDF, from one pair of xacro
properties. Both are 0.7: the old mu2 = 0.3 only has a meaning along a
friction direction (fdir1), which was never set, so the direction it
applied in was up to the physics engine.

Co-Authored-By: Claude Opus 5.5 <noreply@anthropic.com>

* docs: don't refer to what was in the past

---------

Co-authored-by: Claude Opus 5.5 <noreply@anthropic.com>
Co-authored-by: Achille Verheye <achille.verheye@gmail.com>

File: ROS/osr_gazebo/urdf/osr.urdf.xacro (robot description, xacro)
@@ -305,5 +305,17 @@
     <xacro:wheel_link prefix="L" dir="1" origin="1.57"/>
     <xacro:wheel_link prefix="R" dir="-1" origin="-3.14"/>
+    <!-- Wheel-ground friction -->
+    <xacro:property name="wheel_mu1" value="0.7"/>
+    <xacro:property name="wheel_mu2" value="0.7"/>
+    <xacro:macro name="wheel_friction" params="link">
+        <gazebo reference="${link}">
+            <mu1>${wheel_mu1}</mu1>
+            <mu2>${wheel_mu2}</mu2>
+        </gazebo>
+    </xacro:macro>
     <xacro:macro name="wheel" params="prefix dir origin prefix_1">
+        <xacro:wheel_friction link="front_wheel_link_${prefix}"/>
+        <xacro:wheel_friction link="middle_wheel_link_${prefix}"/>
+        <xacro:wheel_friction link="rear_wheel_link_${prefix}"/>
         <link name="front_wheel_link_${prefix}">
             <collision>
@@ -312,12 +324,4 @@
                     <mesh filename="file://$(find osr_gazebo)/meshes/wheel.stl"/>
                 </geometry>
-                <surface>
-                    <friction>
-                        <ode>
-                            <mu>0.7</mu>
-                            <mu2>0.3</mu2>
-                        </ode>
-                    </friction>
-                </surface>
             </collision>
             <visual>
@@ -347,12 +351,4 @@
                     <mesh filename="file://$(find osr_gazebo)/meshes/wheel.stl"/>
                 </geometry>
-                <surface>
-                    <friction>
-                        <ode>
-                            <mu>0.7</mu>
-                            <mu2>0.3</mu2>
-                        </ode>
-                    </friction>
-                </surface>
             </collision>
             <visual>
@@ -382,12 +378,4 @@
                     <mesh filename="file://$(find osr_gazebo)/meshes/wheel.stl"/>
                 </geometry>
-                <surface>
-                    <friction>
-                        <ode>
-                            <mu>0.7</mu>
-                            <mu2>0.3</mu2>
-                        </ode>
-                    </friction>
-                </surface>
             </collision>
             <visual>
